File: ESP32_Development_Board.kicad_sch (KiCad schematic)
At the start: 47 parts, among them J1 Conn_01x17_Pin, J2 Conn_01x17_Pin, J3 Conn_01x03_Pin, J4 USB_B_Micro, J5 Conn_01x02_Pin, Q1 NPN, Q2 NPN, Q3 Q_NMOS_GDS, Q4 Q_NMOS_GDS, SW1 SW_Push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

Commit message: Aug 16, 2025
Parts:
- U3: footprint Package_TO_SOT_SMD:SOT-223-3_TabPin2 -> Package_TO_SOT_SMD:SOT-89-3
Connections:
- net USB_DN: now also D5.2 (A2), J4.2 (D-), Q4.2 (D); no longer D4.2 (A2), J4.3 (D+), Q3.2 (D)
- net USB_DP: now also D4.2 (A2), J4.3 (D+), Q3.2 (D); no longer D5.2 (A2), J4.2 (D-), Q4.2 (D)
Changed lines of the file:
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@@
 		)
 	)
-	(label "USB_DP"
+	(label "USB_DN"
 		(at 236.22 107.95 180)
 		(fields_autoplaced yes)
@@
 		)
 	)
-	(label "USB_DN"
+	(label "USB_DP"
 		(at 236.22 105.41 180)
 		(fields_autoplaced yes)
@@
 			)
 		)
-		(property "Footprint" "Package_TO_SOT_SMD:SOT-223-3_TabPin2"
+		(property "Footprint" "Package_TO_SOT_SMD:SOT-89-3"
 			(at 163.83 22.86 0)
 			(effects
