File: ESP32_Development_Board.kicad_pcb (KiCad board)
At the start: 4 copper layers, 70 x 20.3 mm, 47 parts, among them J1 Conn_01x17_Pin, J2 Conn_01x17_Pin, J3 Conn_01x03_Pin, J4 USB_B_Micro, J5 Conn_01x02_Pin, Q1 NPN, Q2 NPN, Q3 Q_NMOS_GDS, Q4 Q_NMOS_GDS, SW1 SW_Push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

Commit message: Commit at 2025-08-20 20:00:00
Routing:
- net /IO23: track 4.25 -> 65.0 mm
- net /IO22: track 1.86 -> 58.3 mm
- net /TXD0: track 1.86 -> 57.7 mm
- net /RXD0: track 1.86 -> 53.5 mm
- net /IO21: track 1.86 -> 49.7 mm
- net /IO19: track 1.86 -> 41.5 mm
- net /IO18: track 1.86 -> 37.5 mm
- net /IO5: track 1.86 -> 33.4 mm
- net /IO17: track 1.86 -> 28.3 mm
- net /IO16: track 1.86 -> 24.3 mm
- net /IO4: track 1.86 -> 21.1 mm
- net /IO0_BTN: track 2.40 -> 15.8 mm, vias 0 -> 2
- net /IO13: track 0.00 -> 11.6 mm, vias 0 -> 1
- net /IO15: track 0.00 -> 11.3 mm
- net /IO2: track 0.00 -> 10.1 mm
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
Commit message: Commit at 2025-08-20 22:00:00
Parts:
- moved R3 0.79 mm to (121.3, 92.0)
- moved C3 0.78 mm to (121.3, 94.0)
Routing:
- net +5VA: track 5.74 -> 43.2 mm, vias 1 -> 2
- net /IO0_BTN: track 15.8 -> 43.6 mm, vias 2 -> 3
- net Net-(Q1-B): track 0.00 -> 24.4 mm, vias 0 -> 2
- net /EN: track 68.7 -> 90.9 mm, vias 1 -> 2
- net /TXD0: track 57.7 -> 77.2 mm
- net /RXD0: track 53.5 -> 71.4 mm
- net Net-(Q2-B): track 0.00 -> 14.9 mm, vias 0 -> 2
- net /IO18: track 37.5 -> 46.5 mm, vias 1 -> 2
- net GND: track 48.8 -> 57.1 mm
- net /RTS: track 4.72 -> 6.03 mm
- net +3.3V: track 26.6 -> 27.5 mm, vias 10 -> 11
- net /IO5: track 33.4 -> 32.5 mm
